File: PCB.kicad_pcb (KiCad board)
At the start: 4 copper layers, 131.4 x 64.3 mm, 31 parts, among them J1 Conn_ARM_SWD_TagConnect_TC2030, U2 STM32L476RGTx, U3 NT3H2X11, U4 SSD1306

Commit message: Add battery as main power source
Do not use NFC power harvesting, update components correspondingly
Parts:
- removed R2, R3: 10k, Resistor_SMD:R_0603_1608Metric
- added BT1: CR2430 3V, Battery:BatteryHolder_Keystone_105_1x2430, B.Cu at (82.3, 140.0)
- R1: value 10k -> 3k
- U2: value STM32L476RGTx -> STM32L476RGT6
- U3: value NT3H2X11 -> NT3H2111W0FT1X
- U4: value SSD1306 -> ER-OLED0.96-1W
- moved R1 1.89 mm to (121.3, 117.3), turned to -90 degrees
- moved R10 1.74 mm to (124.3, 117.3), turned to -90 degrees
Connections:
- R1 pad 1: NFC_SDA -> VCC
- R1 pad 2: VCC -> NFC_INT
- U3 pad 7: VCC -> /NFC_IC/NFC_VOUT
Routing:
- net GND: track 40.8 -> 79.5 mm
- net VCC: track 79.9 -> 105.6 mm, vias 17 -> 16
- net NFC_INT: track 24.2 -> 26.9 mm
- net NFC_SCL: track 19.9 -> 17.5 mm, vias 3 -> 2
- net /NFC_IC/NFC_VOUT: track 0.00 -> 1.51 mm, vias 0 -> 1
- net NFC_SDA: track 21.7 -> 20.9 mm
Other:
- outline, holes or cut-outs redrawn
- board text added: "Board Rev 3 08/15/2026"
- board text removed: "Board Rev 2D 04/20/2024"
