File: PCB.kicad_sch (KiCad schematic)
At the start: 13 parts, among them J1 Conn_ARM_SWD_TagConnect_TC2030, U2 STM32L476RGT6

Commit message: Add battery as main power source
Do not use NFC power harvesting, update components correspondingly
Other:
- note added: "Power Supply"
