File: nfc_ic.kicad_sch (KiCad schematic)
At the start: 7 parts, among them U3 NT3H2111W0FT1X

Commit message: Add battery as main power source
Do not use NFC power harvesting, update components correspondingly
Parts:
- removed R1, R2: 10k, Resistor_SMD:R_0603_1608Metric, symbol Device:R_Small
- R1: renamed from R3; value 10k -> 3k
Connections:
- net NFC_INT: now also R1.2; no longer R1.1
- net VCC: now also R1.1; no longer R1.2, U3.7 (VOUT)
- new net NFC_VOUT: U3.7 (VOUT)
- no-connect marks 0 -> 1
Other:
- moved on the sheet: A1, C18, C8, R1, U3
